File: v2/assemble/assemble.kicad_pcb (KiCad board)
At the start: 2 copper layers, 259.2 x 98.4 mm, 126 parts, among them J1 Conn_01x04, J2 Conn_01x04, J3 Conn_01x04, J4 Conn_01x04, SW1 SW_Push, SW10 SW_Push, SW11 SW_Push, SW12 SW_Push, SW13 SW_Push, SW14 SW_Push, SW15 SW_Push, SW16 SW_Push, SW17 SW_Push, SW18 SW_Push, SW19 SW_Push, SW2 SW_Push, SW20 SW_Push, SW21 SW_Push, SW22 SW_Push, SW23 SW_Push, SW24 SW_Push, SW25 SW_Push, SW26 SW_Push, SW27 SW_Push, SW28 SW_Push, SW29 SW_Push, SW3 SW_Push, SW30 SW_Push, SW31 SW_Push, SW32 SW_Push, SW33 SW_Push, SW34 SW_Push, SW35 SW_Push, SW36 SW_Push, SW37 SW_Push, SW38 SW_Push, SW39 SW_Push, SW4 SW_Push, SW40 SW_Push, SW41 SW_Push, SW42 SW_Push, SW43 SW_SPDT, SW44 SW_SPDT, SW45 RotaryEncoder_Switch, SW46 RotaryEncoder_Switch, SW5 SW_Push, SW6 SW_Push, SW7 SW_Push, SW8 SW_Push, SW9 SW_Push, U1 XIAO-nRF52840-SMD, U2 XIAO-nRF52840-SMD

Commit message: feat: implement v2 assemble
Parts:
- removed BT3, BT4: Battery_Cell, kbd_Parts:Battery_AAA
- added Q1: DMG3414U, Package_TO_SOT_SMD:SOT-23, B.Cu at (135.7, 75.7)
- added Q2: DMG3414U, Package_TO_SOT_SMD:SOT-23, B.Cu at (159.6, 75.7)
- added R10: 1M, Resistor_SMD:R_0805_2012Metric_Pad1.20x1.40mm_HandSolder, B.Cu at (142.8, 59.3)
- added R11: 470k, Resistor_SMD:R_0805_2012Metric_Pad1.20x1.40mm_HandSolder, B.Cu at (165.0, 59.3)
- added R12: 1M, Resistor_SMD:R_0805_2012Metric_Pad1.20x1.40mm_HandSolder, B.Cu at (168.4, 59.3)
- added R5: 470k, Resistor_SMD:R_0805_2012Metric_Pad1.20x1.40mm_HandSolder, B.Cu at (164.3, 69.9)
- added R6: 22k, Resistor_SMD:R_0805_2012Metric_Pad1.20x1.40mm_HandSolder, B.Cu at (165.1, 53.6)
- added R7: 22k, Resistor_SMD:R_0805_2012Metric_Pad1.20x1.40mm_HandSolder, B.Cu at (139.5, 53.6)
- added R8: 470k, Resistor_SMD:R_0805_2012Metric_Pad1.20x1.40mm_HandSolder, B.Cu at (139.5, 70.0)
- added R9: 470k, Resistor_SMD:R_0805_2012Metric_Pad1.20x1.40mm_HandSolder, B.Cu at (139.4, 59.3)
- added Ref**: Val**, kbd_Hole:m2_Screw_Hole, F.Cu at (66.7, 45.3)
- added Ref**: Val**, kbd_Hole:m2_Screw_Hole, F.Cu at (236.3, 45.3)
- J1, J3: value Conn_01x04 -> Conn_01x03; footprint Connector_JST:JST_ZH_B4B-ZR_1x04_P1.50mm_Vertical -> Connector_JST:JST_ZH_B3B-ZR_1x03_P1.50mm_Vertical; moved to F.Cu
- J2, J4: value Conn_01x04 -> Conn_01x03; footprint Connector_JST:JST_ZH_B4B-ZR_1x04_P1.50mm_Vertical -> Connector_JST:JST_ZH_B3B-ZR_1x03_P1.50mm_Vertical
- moved J1 28.2 mm to (165.0, 75.2)
- moved J2 23.3 mm to (160.7, 44.8)
- moved J3 22.0 mm to (140.9, 75.2)
- moved J4 21.8 mm to (139.3, 44.8)
- moved D5 7.46 mm to (174.3, 78.7)
- moved D6 7.46 mm to (174.3, 81.6)
- moved D7 7.46 mm to (174.3, 84.5)
- moved D8 7.46 mm to (174.3, 87.4)
- moved D2 7.31 mm to (129.4, 84.1)
- moved D1 7.31 mm to (129.4, 87.0)
- moved D3 7.31 mm to (129.4, 81.2)
- moved D4 7.31 mm to (129.4, 78.3)
- moved BT2 4.20 mm to (72.8, 40.6)
- moved BT1 2.21 mm to (230.2, 40.5), turned to 180 degrees
- moved SW43 1.31 mm to (172.9, 34.8)
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Connections:
- AE-XCL102D333CR-G1 pad 6: Net-(BT3-+) -> Net-(BT1-+)
- AE-XCL102D333CR-G2 pad 6: Net-(BT4-+) -> Net-(BT2-+)
- J1 pad 1: B+L -> Net-(J1-Pin_1)
- J1 pad 2: BAT+L -> Net-(J1-Pin_2)
- J1 pad 3: BAT-L -> GNDR
- J2 pad 1: Net-(BT4-+) -> Net-(BT1-+)
- J2 pad 2: Net-(AE-XCL102D333CR-G2-OUT) -> Net-(AE-XCL102D333CR-G1-OUT)
- J2 pad 3: Net-(BT2--) -> Net-(BT1--)
- J3 pad 1: B+R -> Net-(J3-Pin_1)
- J3 pad 2: BAT+R -> Net-(J3-Pin_2)
- J3 pad 3: BAT-R -> GNDL
- J4 pad 1: Net-(BT3-+) -> Net-(BT2-+)
- J4 pad 2: Net-(AE-XCL102D333CR-G1-OUT) -> Net-(AE-XCL102D333CR-G2-OUT)
- J4 pad 3: Net-(BT1--) -> Net-(BT2--)
- U1 pad 1: RE1A -> B+L
- U1 pad 12: VCCL -> BAT+L
- U1 pad 14: unconnected-(U1-5V-Pad14) -> 5V-L
- U1 pad 2: RE1B -> RE1A
- U1 pad 3: B+L -> RE1B
- U2 pad 1: RE2A -> B+R
- U2 pad 12: VCCR -> BAT+R
- U2 pad 14: unconnected-(U2-5V-Pad14) -> 5V-R
- U2 pad 2: RE2B -> RE2A
- U2 pad 3: B+R -> RE2B
Routing:
- net Net-(D18-A): track 0.00 -> 217.8 mm, vias 0 -> 22
- net Net-(D17-A): track 0.00 -> 214.8 mm, vias 0 -> 15
- net Net-(D1-A): track 0.00 -> 207.5 mm, vias 0 -> 7
- net Net-(D25-A): track 0.00 -> 193.5 mm, vias 0 -> 14
- net Net-(D10-A): track 0.00 -> 191.0 mm, vias 0 -> 16
- net Net-(D26-A): track 0.00 -> 181.0 mm, vias 0 -> 15
- net PIN1L: track 0.00 -> 169.8 mm, vias 0 -> 10
- net PIN6R: track 0.00 -> 153.9 mm, vias 0 -> 7
- net PIN2L: track 0.00 -> 153.0 mm, vias 0 -> 9
- net PIN4L: track 0.00 -> 142.8 mm, vias 0 -> 8
- net PIN5R: track 0.00 -> 141.1 mm, vias 0 -> 8
- net PIN4R: track 0.00 -> 140.3 mm, vias 0 -> 8
- net Net-(D33-A): track 0.44 -> 131.8 mm, vias 0 -> 9
- net PIN3L: track 0.00 -> 114.8 mm, vias 0 -> 9
- net PIN5L: track 0.00 -> 113.7 mm, vias 0 -> 6
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Other:
- board size 259.2 x 98.4 mm -> 252.6 x 98.4 mm
