File: v2/assemble/assemble.kicad_sch (KiCad schematic)
At the start: 124 parts, among them J1 Conn_01x04, J2 Conn_01x04, J3 Conn_01x04, J4 Conn_01x04, SW1 SW_Push, SW10 SW_Push, SW11 SW_Push, SW12 SW_Push, SW13 SW_Push, SW14 SW_Push, SW15 SW_Push, SW16 SW_Push, SW17 SW_Push, SW18 SW_Push, SW19 SW_Push, SW2 SW_Push, SW20 SW_Push, SW21 SW_Push, SW22 SW_Push, SW23 SW_Push, SW24 SW_Push, SW25 SW_Push, SW26 SW_Push, SW27 SW_Push, SW28 SW_Push, SW29 SW_Push, SW3 SW_Push, SW30 SW_Push, SW31 SW_Push, SW32 SW_Push, SW33 SW_Push, SW34 SW_Push, SW35 SW_Push, SW36 SW_Push, SW37 SW_Push, SW38 SW_Push, SW39 SW_Push, SW4 SW_Push, SW40 SW_Push, SW41 SW_Push, SW42 SW_Push, SW43 SW_SPDT, SW44 SW_SPDT, SW45 RotaryEncoder_Switch, SW46 RotaryEncoder_Switch, SW5 SW_Push, SW6 SW_Push, SW7 SW_Push, SW8 SW_Push, SW9 SW_Push, U1 XIAO-nRF52840-SMD, U2 XIAO-nRF52840-SMD

Commit message: refactor: move files
Parts:
- AE-XCL102D333CR-G1, AE-XCL102D333CR-G2: value ~ -> (none)
- C1, C2, C3, C4: value 0.01uF -> 0.1uF; footprint kbd_Parts:Capacitor_1206 -> Capacitor_SMD:C_0603_1608Metric_Pad1.08x0.95mm_HandSolder
- J2, J4: footprint Connector_Wire:SolderWire-0.5sqmm_1x04_P4.6mm_D0.9mm_OD2.1mm -> Connector_JST:JST_ZH_B4B-ZR_1x04_P1.50mm_Vertical
- R1, R2, R3, R4: value 10K -> 2.2K
Connections:
- net B+L: no longer AE-XCL102D333CR-G2.6 (IN)
- net B+R: no longer AE-XCL102D333CR-G1.6 (IN)
- net BAT+L: now also J1.2 (Pin_2); no longer AE-XCL102D333CR-G2.4 (OUT)
- net BAT+R: now also J3.2 (Pin_2); no longer AE-XCL102D333CR-G1.4 (OUT)
- net at BT3.1 (+), J4.1 (Pin_1): now also AE-XCL102D333CR-G1.6 (IN)
- net at J4.2 (Pin_2): now also AE-XCL102D333CR-G1.4 (OUT); no longer BT1.2 (-)
- net at J4.3 (Pin_3): now also AE-XCL102D333CR-G1.5 (GND), BT1.2 (-); no longer SW43.3 (C)
- net at J4.4 (Pin_4): no longer SW43.2 (B)
- net at BT4.1 (+), J2.1 (Pin_1): now also AE-XCL102D333CR-G2.6 (IN)
- net at J2.2 (Pin_2): now also AE-XCL102D333CR-G2.4 (OUT); no longer BT2.2 (-)
- net at J2.3 (Pin_3): now also AE-XCL102D333CR-G2.5 (GND), BT2.2 (-); no longer SW44.3 (C)
- net at J2.4 (Pin_4): no longer SW44.2 (B)
- net at AE-XCL102D333CR-G2.2 (EN): now also SW44.2 (B); no longer J1.4 (Pin_4)
- net at AE-XCL102D333CR-G2.3 (GND): now also SW44.3 (C); no longer J1.3 (Pin_3)
- net at AE-XCL102D333CR-G1.3 (GND): now also SW43.3 (C); no longer J3.3 (Pin_3)
- net at AE-XCL102D333CR-G1.2 (EN): now also SW43.2 (B); no longer J3.4 (Pin_4)
- removed net B-L: AE-XCL102D333CR-G2.5 (GND), J1.2 (Pin_2), U1.16 (GND)
- removed net B-R: AE-XCL102D333CR-G1.5 (GND), J3.2 (Pin_2), U2.16 (GND)
- new net BAT-L: J1.3 (Pin_3), U1.16 (GND)
- new net BAT-R: J3.3 (Pin_3), U2.16 (GND)
- no-connect marks 22 -> 26
Other:
- moved on the sheet: AE-XCL102D333CR-G2, BT1, BT3, J1, J2, J3, J4, SW43, SW44

Commit message: feat: implement v2 assemble
Parts:
- removed BT3, BT4: Battery_Cell, kbd_Parts:Battery_AAA, symbol Device:Battery_Cell
- removed J1, J2, J3, J4: Conn_01x04, Connector_JST:JST_ZH_B4B-ZR_1x04_P1.50mm_Vertical, symbol Connector_Generic:Conn_01x04
- added J1, J2, J3, J4: Conn_01x03, Connector_JST:JST_ZH_B3B-ZR_1x03_P1.50mm_Vertical, symbol Connector_Generic:Conn_01x03
- added Q1, Q2: DMG3414U, Package_TO_SOT_SMD:SOT-23, symbol Transistor_FET:DMG3414U
- added R10, R12: 1M, Resistor_SMD:R_0805_2012Metric_Pad1.20x1.40mm_HandSolder, symbol Device:R
- added R11, R5, R8, R9: 470k, Resistor_SMD:R_0805_2012Metric_Pad1.20x1.40mm_HandSolder, symbol Device:R
- added R6, R7: 22k, Resistor_SMD:R_0805_2012Metric_Pad1.20x1.40mm_HandSolder, symbol Device:R
Connections:
- net VCCL is gone; now on net BAT+L: U1.12 (3V3)
- net VCCR is gone; now on net BAT+R: U2.12 (3V3)
- net B+L: now also U1.1 (P0.02_A0_D0), R10.2, R9.1; no longer U1.3 (P0.28_A2_D2)
- net B+R: now also U2.1 (P0.02_A0_D0), R11.1, R12.1; no longer U2.3 (P0.28_A2_D2)
- net BAT+L: now also Q1.3 (D); no longer U1.15 (BAT)
- net BAT+R: now also Q2.3 (D); no longer U2.15 (BAT)
- net GNDL: now also J3.3 (Pin_3), R10.1, R8.1
- net GNDR: now also J1.3 (Pin_3), R12.2, R5.1
- net RE1A: now also U1.2 (P0.03_A1_D1); no longer U1.1 (P0.02_A0_D0)
- net RE1B: now also U1.3 (P0.28_A2_D2); no longer U1.2 (P0.03_A1_D1)
- net RE2A: now also U2.2 (P0.03_A1_D1); no longer U2.1 (P0.02_A0_D0)
- net RE2B: now also U2.3 (P0.28_A2_D2); no longer U2.2 (P0.03_A1_D1)
- net 5V-L: now reaches U1.14 (5V)
- net 5V-L: now also R7.2
- net at AE-XCL102D333CR-G1.6 (IN): now also BT1.1 (+), J2.1 (Pin_1)
- net at AE-XCL102D333CR-G1.4 (OUT): now also J2.2 (Pin_2)
- net at AE-XCL102D333CR-G1.5 (GND), BT1.2 (-): now also J2.3 (Pin_3)
- net at AE-XCL102D333CR-G2.6 (IN): now also BT2.1 (+), J4.1 (Pin_1)
- net at AE-XCL102D333CR-G2.4 (OUT): now also J4.2 (Pin_2)
- net at AE-XCL102D333CR-G2.5 (GND), BT2.2 (-): now also J4.3 (Pin_3)
- net 5V-R: now reaches U2.14 (5V)
- net 5V-R: now also R6.2
- net BAT-L: no longer names the net of U1.16 (GND)
- net BAT-R: no longer names the net of U2.16 (GND)
- new net: Q1.1 (G), R7.1, R8.2
- new net: Q2.1 (G), R5.2, R6.1
- new net: J1.2 (Pin_2), Q2.2 (S)
- new net: J1.1 (Pin_1), R11.2
- new net: J3.1 (Pin_1), R9.2
- new net: J3.2 (Pin_2), Q1.2 (S)
- no-connect marks 26 -> 24
Other:
- moved on the sheet: AE-XCL102D333CR-G1, AE-XCL102D333CR-G2, BT1, BT2, SW43, SW44
